File: vdg_voltage_sensor_rev2.brd (EAGLE design)
At the start: 35.7 x 46.9 mm, 8 parts, among them J1 VANDEGRAAFF, U1 ADS1100A0IDBVRDBV6-M

Commit message: Added full wiring diagram
Added full wiring diagram and an image.
Parts:
- C1: value 2uF -> 3uf
Changed lines of the file:
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@@
 </autorouter>
 <elements>
-<element name="C1" library="Resistor_Capacitor" library_urn="urn:adsk.eagle:library:15122775" package="CAP_1206" package3d_urn="urn:adsk.eagle:package:10872907/3" value="2uF" x="6.53" y="17.09" rot="R90">
+<element name="C1" library="Resistor_Capacitor" library_urn="urn:adsk.eagle:library:15122775" package="CAP_1206" package3d_urn="urn:adsk.eagle:package:10872907/3" value="3uf" x="6.53" y="17.09" rot="R90">
 <attribute name="CREATED_BY" value="PCBLayout.com" x="25.58" y="46.3" size="1.778" layer="27" rot="R90" display="off"/>
 <attribute name="DIGIKEY_PART_NUMBER" value="GRM31CR60J107ME39L" x="25.58" y="46.3" size="1.778" layer="27" rot="R90" display="off"/>
